Commit message: 引入gazobo,ros2

File: src/piper_description/urdf/piper_gazebo.urdf (robot description, URDF)
Before this commit: robot piper, 10 links, 9 joints
Links:
- link base_link: geometry collision cylinder length=0.05 radius=0.06; visual mesh filename=package://piper_description/meshes/base_link.stl
- link link1: geometry collision cylinder length=0.12 radius=0.035; visual mesh filename=package://piper_description/meshes/link1.stl
- link link2: geometry collision cylinder length=0.28 radius=0.03; visual mesh filename=package://piper_description/meshes/link2.stl
- link link3: geometry collision cylinder length=0.24 radius=0.025; visual mesh filename=package://piper_description/meshes/link3.stl
- link link4: geometry collision cylinder length=0.1 radius=0.025; visual mesh filename=package://piper_description/meshes/link4.stl
- link link5: geometry collision cylinder length=0.09 radius=0.02; visual mesh filename=package://piper_description/meshes/link5.stl
- link link6: geometry collision cylinder length=0.06 radius=0.035; visual mesh filename=package://piper_description/meshes/link6.stl
- link link7: geometry collision box size=0.02 0.04 0.02; visual mesh filename=package://piper_description/meshes/link7.stl
- link link8: geometry collision box size=0.02 0.04 0.02; visual mesh filename=package://piper_description/meshes/link8.stl
- link wrist_cam_link: geometry collision box size=0.028 0.034 0.024; visual box size=0.028 0.034 0.024
