Commit message: 修复了真机bug
Co-authored-by: Copilot <copilot@github.com>

File: src/piper_description/urdf/piper.ros2_control.xacro (robot description, xacro)
@@ -48,6 +48,8 @@
           <param name="initial_value">${initial_positions['joint1']}</param>
         </state_interface>
-        <state_interface name="velocity"/>
-        <state_interface name="effort"/>
+        <xacro:unless value="${real_hardware}">
+          <state_interface name="velocity"/>
+          <state_interface name="effort"/>
+        </xacro:unless>
       </joint>
       <joint name="${prefix}joint2">
@@ -59,10 +61,12 @@
           <param name="initial_value">${initial_positions['joint2']}</param>
         </state_interface>
-        <state_interface name="velocity"/>
-        <state_interface name="effort"/>
+        <xacro:unless value="${real_hardware}">
+          <state_interface name="velocity"/>
+          <state_interface name="effort"/>
+        </xacro:unless>
       </joint>
       <joint name="${prefix}joint3">
         <command_interface name="position">
-          <param name="min">-2.967</param>
+          <param name="min">-2.697</param>
           <param name="max">0</param>
         </command_interface>
@@ -70,6 +74,8 @@
           <param name="initial_value">${initial_positions['joint3']}</param>
         </state_interface>
-        <state_interface name="velocity"/>
-        <state_interface name="effort"/>
+        <xacro:unless value="${real_hardware}">
+          <state_interface name="velocity"/>
+          <state_interface name="effort"/>
+        </xacro:unless>
       </joint>
       <joint name="${prefix}joint4">
@@ -81,6 +87,8 @@
           <param name="initial_value">${initial_positions['joint4']}</param>
         </state_interface>
-        <state_interface name="velocity"/>
-        <state_interface name="effort"/>
+        <xacro:unless value="${real_hardware}">
+          <state_interface name="velocity"/>
+          <state_interface name="effort"/>
+        </xacro:unless>
       </joint>
       <joint name="${prefix}joint5">
@@ -92,6 +100,8 @@
           <param name="initial_value">${initial_positions['joint5']}</param>
         </state_interface>
-        <state_interface name="velocity"/>
-        <state_interface name="effort"/>
+        <xacro:unless value="${real_hardware}">
+          <state_interface name="velocity"/>
+          <state_interface name="effort"/>
+        </xacro:unless>
       </joint>
       <joint name="${prefix}joint6">
@@ -103,6 +113,8 @@
           <param name="initial_value">${initial_positions['joint6']}</param>
         </state_interface>
-        <state_interface name="velocity"/>
-        <state_interface name="effort"/>
+        <xacro:unless value="${real_hardware}">
+          <state_interface name="velocity"/>
+          <state_interface name="effort"/>
+        </xacro:unless>
       </joint>
       <xacro:if value="${include_gripper}">
@@ -112,6 +124,8 @@
             <param name="initial_value">0.0</param>
           </state_interface>
-          <state_interface name="velocity"/>
-          <state_interface name="effort"/>
+          <xacro:unless value="${real_hardware}">
+            <state_interface name="velocity"/>
+            <state_interface name="effort"/>
+          </xacro:unless>
         </joint>
       </xacro:if>

File: src/piper_description/urdf/piper_arm_macro.xacro (robot description, xacro)
@@ -87,5 +87,5 @@
     </link>
     <joint name="${prefix}joint2" type="revolute">
-      <origin xyz="0 0 0" rpy="${pi/2} -0.10095 -${pi/2}" />
+      <origin xyz="0 0 0" rpy="${pi/2} 0 -${pi/2}" />
       <parent link="${prefix}link_1" />
       <child link="${prefix}link_2" />
@@ -117,9 +117,9 @@
     </link>
     <joint name="${prefix}joint3" type="revolute">
-      <origin xyz="0.28503 0 0" rpy="0 0 1.3826" />
+      <origin xyz="0.28358 0.028726 0" rpy="0 0 0.1009" />
       <parent link="${prefix}link_2" />
       <child link="${prefix}link_3" />
       <axis xyz="0 0 1" />
-      <limit lower="-3.0" upper="0" effort="100" velocity="3.14" />
+      <limit lower="-2.697" upper="0" effort="100" velocity="3.14" />
     </joint>
     <link name="${prefix}link_4">
@@ -147,8 +147,8 @@
     </link>
     <joint name="${prefix}joint4" type="revolute">
-      <origin xyz="0.021984 0.25075 0" rpy="-${pi/2} 0 0" />
+      <origin xyz="-0.24221 0.068514 0" rpy="-${pi/2} 0 1.382" />
       <parent link="${prefix}link_3" />
       <child link="${prefix}link_4" />
-      <axis xyz="0 0 -1" />
+      <axis xyz="0 0 1" />
       <limit lower="-1.85" upper="1.85" effort="100" velocity="3.93" />
     </joint>
@@ -177,5 +177,5 @@
     </link>
     <joint name="${prefix}joint5" type="revolute">
-      <origin xyz="0 0 0" rpy="${pi/2} -0.087266 0" />
+      <origin xyz="0 0 0" rpy="${pi/2} 0 0" />
       <parent link="${prefix}link_4" />
       <child link="${prefix}link_5" />
@@ -183,10 +183,31 @@
       <limit lower="-1.3" upper="1.3" effort="100" velocity="3.93" />
     </joint>
-    <link name="${prefix}link_6" />
+    <link name="${prefix}link_6">
+      <inertial>
+        <origin xyz="0.00103 0.01218 0.03155" rpy="0 0 0" />
+        <mass value="1.2" />
+        <inertia
+          ixx="0.001" ixy="0" ixz="0"
+          iyy="0.001" iyz="0"
+          izz="0.001" />
+      </inertial>
+      <visual>
+        <origin xyz="0 0 0" rpy="0 0 ${pi/2}" />
+        <geometry>
+          <mesh filename="file://$(find piper_description)/meshes/link6.stl" />
+        </geometry>
+      </visual>
+      <collision>
+        <origin xyz="0 0 0" rpy="0 0 ${pi/2}" />
+        <geometry>
+          <mesh filename="file://$(find piper_description)/meshes/link6.stl" />
+        </geometry>
+      </collision>
+    </link>
     <joint name="${prefix}joint6" type="revolute">
-      <origin xyz="0 0.091 0.0014" rpy="-${pi/2} 0 0" />
+      <origin xyz="0 0.091 0.0014165" rpy="${pi/2} 0 ${pi}" />
       <parent link="${prefix}link_5" />
       <child link="${prefix}link_6" />
-      <axis xyz="0 0 -1" />
+      <axis xyz="0 0 1" />
       <limit lower="-${pi}" upper="${pi}" effort="100" velocity="3.93" />
     </joint>

File: src/piper_description/urdf/piper_gripper_macro.xacro (robot description, xacro)
@@ -5,4 +5,6 @@
     prefix
     *origin">
+    <!-- 夹爪基座：与官方 piper.xml 对齐，仅作为坐标系（link6 沿其 z 轴偏移 0.13503m）。
+         夹爪本体外形已包含在 link6.stl 中，此处不再放置占位方块。 -->
     <joint name="${prefix}gripper_base_joint" type="fixed">
       <xacro:insert_block name="origin" />
@@ -16,25 +18,12 @@
         <inertia ixx="0.0001" ixy="0" ixz="0" iyy="0.0001" iyz="0" izz="0.0001" />
       </inertial>
-      <visual>
-        <origin xyz="0 0 0" rpy="0 0 0" />
-        <geometry>
-          <box size="0.06 0.04 0.04"/>
-        </geometry>
-        <material name="gripper_body_mat">
-          <color rgba="0.9 0.7 0.1 1"/>
-        </material>
-      </visual>
-      <collision>
-        <origin xyz="0 0 0" rpy="0 0 0" />
-        <geometry>
-          <box size="0.06 0.04 0.04"/>
-        </geometry>
-      </collision>
     </link>
+    <!-- 左指 (link7)：相对 link6 的变换 quat=(0,0,0.7071,0.7071) → rpy=(pi/2,0,pi)，
+         沿指尖局部 -z 滑动，行程 0~0.035m（对应 piper.xml joint7）。 -->
     <joint name="${prefix}gripper_joint" type="prismatic">
-      <origin xyz="0 0.047 0" rpy="0 0 0" />
+      <origin xyz="0 0 0" rpy="${pi/2} 0 ${pi}" />
       <parent link="${prefix}gripper_base_link"/>
       <child link="${prefix}left_finger"/>
-      <axis xyz="0 1 0" />
+      <axis xyz="0 0 -1" />
       <limit lower="0" upper="0.035" effort="20" velocity="0.1" />
     </joint>
@@ -48,5 +37,5 @@
         <origin xyz="0 0 0" rpy="0 0 0" />
         <geometry>
-          <box size="0.02 0.01 0.04"/>
+          <mesh filename="file://$(find piper_description)/meshes/link7.stl" />
         </geometry>
         <material name="finger_mat">
@@ -57,14 +46,17 @@
         <origin xyz="0 0 0" rpy="0 0 0" />
         <geometry>
-          <box size="0.02 0.01 0.04"/>
+          <mesh filename="file://$(find piper_description)/meshes/link7.stl" />
         </geometry>
       </collision>
     </link>
+    <!-- 右指 (link8)：quat=(0,0,-0.7071,0.7071) → rpy=(-pi/2,0,pi)，沿局部 +z 滑动。
+         mimic 左指、系数 -1（对应 piper.xml equality joint8 = -joint7），行程 -0.035~0。 -->
     <joint name="${prefix}right_finger_joint" type="prismatic">
-      <origin xyz="0 -0.047 0" rpy="0 0 0" />
+      <origin xyz="0 0 0" rpy="-${pi/2} 0 ${pi}" />
       <parent link="${prefix}gripper_base_link"/>
       <child link="${prefix}right_finger"/>
-      <axis xyz="0 -1 0" />
-      <limit lower="0" upper="0.035" effort="20" velocity="0.1" />
+      <axis xyz="0 0 1" />
+      <limit lower="-0.035" upper="0" effort="20" velocity="0.1" />
+      <mimic joint="${prefix}gripper_joint" multiplier="-1" offset="0" />
     </joint>
     <link name="${prefix}right_finger">
@@ -77,5 +69,5 @@
         <origin xyz="0 0 0" rpy="0 0 0" />
         <geometry>
-          <box size="0.02 0.01 0.04"/>
+          <mesh filename="file://$(find piper_description)/meshes/link8.stl" />
         </geometry>
         <material name="finger_mat">
@@ -86,5 +78,5 @@
         <origin xyz="0 0 0" rpy="0 0 0" />
         <geometry>
-          <box size="0.02 0.01 0.04"/>
+          <mesh filename="file://$(find piper_description)/meshes/link8.stl" />
         </geometry>
       </collision>

File: src/piper_moveit_config/config/piper.srdf.xacro (robot description, xacro)
@@ -5,7 +5,6 @@
     </group>
     <group name="gripper">
-        <link name="gripper_base_link"/>
+        <chain base_link="gripper_base_link" tip_link="left_finger"/>
         <link name="right_finger"/>
-        <link name="left_finger"/>
     </group>
     <!-- home pose is just off the joint limits for joint2/3 to keep it from getting stuck in Gazebo simulation -->
@@ -27,5 +26,5 @@
     </group_state>
     <group_state name="open" group="gripper">
-        <joint name="gripper_joint" value="0.038"/>
+        <joint name="gripper_joint" value="0.035"/>
     </group_state>
     <group_state name="closed" group="gripper">
@@ -35,26 +34,29 @@
     <end_effector name="eff" parent_link="tool_0" group="gripper" parent_group="manipulator"/>
     <!--DISABLE COLLISIONS: By default it is assumed that any link of the robot could potentially come into collision with any other link in the robot. This tag disables collision checking between a specified pair of links. -->
-    <disable_collisions link1="base_link" link2="link1" reason="Adjacent"/>
-    <disable_collisions link1="base_link" link2="link2" reason="Never"/>
+    <disable_collisions link1="base_link" link2="link_1" reason="Adjacent"/>
+    <disable_collisions link1="base_link" link2="link_2" reason="Never"/>
     <disable_collisions link1="base_link" link2="table" reason="Adjacent"/>
     <disable_collisions link1="gripper_base_link" link2="left_finger" reason="Adjacent"/>
-    <disable_collisions link1="gripper_base_link" link2="link3" reason="Never"/>
-    <disable_collisions link1="gripper_base_link" link2="link4" reason="Never"/>
-    <disable_collisions link1="gripper_base_link" link2="link5" reason="Adjacent"/>
+    <disable_collisions link1="gripper_base_link" link2="link_3" reason="Never"/>
+    <disable_collisions link1="gripper_base_link" link2="link_4" reason="Never"/>
+    <disable_collisions link1="gripper_base_link" link2="link_5" reason="Adjacent"/>
+    <disable_collisions link1="gripper_base_link" link2="link_6" reason="Adjacent"/>
     <disable_collisions link1="gripper_base_link" link2="right_finger" reason="Adjacent"/>
-    <disable_collisions link1="left_finger" link2="link3" reason="Never"/>
-    <disable_collisions link1="left_finger" link2="link4" reason="Never"/>
-    <disable_collisions link1="left_finger" link2="link5" reason="Never"/>
+    <disable_collisions link1="left_finger" link2="link_3" reason="Never"/>
+    <disable_collisions link1="left_finger" link2="link_4" reason="Never"/>
+    <disable_collisions link1="left_finger" link2="link_5" reason="Never"/>
     <disable_collisions link1="left_finger" link2="right_finger" reason="Default"/>
-    <disable_collisions link1="link1" link2="link2" reason="Adjacent"/>
-    <disable_collisions link1="link1" link2="link3" reason="Never"/>
-    <disable_collisions link1="link1" link2="table" reason="Never"/>
-    <disable_collisions link1="link2" link2="link3" reason="Adjacent"/>
-    <disable_collisions link1="link2" link2="link4" reason="Never"/>
-    <disable_collisions link1="link3" link2="link4" reason="Adjacent"/>
-    <disable_collisions link1="link3" link2="link5" reason="Never"/>
-    <disable_collisions link1="link3" link2="right_finger" reason="Never"/>
-    <disable_collisions link1="link4" link2="link5" reason="Adjacent"/>
-    <disable_collisions link1="link4" link2="right_finger" reason="Never"/>
-    <disable_collisions link1="link5" link2="right_finger" reason="Never"/>
+    <disable_collisions link1="link_1" link2="link_2" reason="Adjacent"/>
+    <disable_collisions link1="link_1" link2="link_3" reason="Never"/>
+    <disable_collisions link1="link_1" link2="table" reason="Never"/>
+    <disable_collisions link1="link_2" link2="link_3" reason="Adjacent"/>
+    <disable_collisions link1="link_2" link2="link_4" reason="Never"/>
+    <disable_collisions link1="link_3" link2="link_4" reason="Adjacent"/>
+    <disable_collisions link1="link_3" link2="link_5" reason="Never"/>
+    <disable_collisions link1="link_3" link2="right_finger" reason="Never"/>
+    <disable_collisions link1="link_4" link2="link_5" reason="Adjacent"/>
+    <disable_collisions link1="link_4" link2="right_finger" reason="Never"/>
+    <disable_collisions link1="link_5" link2="right_finger" reason="Never"/>
+    <disable_collisions link1="link_6" link2="left_finger" reason="Default"/>
+    <disable_collisions link1="link_6" link2="right_finger" reason="Default"/>
 </robot>
