Commit message: 新增OrbbecSDK子模块和docker compose多环境配置 2.优化控制器参数、URDF关节限制与

File: src/piper_description/urdf/piper.ros2_control.xacro (robot description, xacro)
@@ -6,7 +6,13 @@
     include_gripper:=true
     mock_hardware:=false
-    fake_sensor_commands:=false
     sim_mujoco:=false
     real_hardware:=false
+    calibration_mode:=false
+    can_interface:=can0
+    speed_percent:=20
+    feedback_timeout_ms:=250
+    max_arm_step:=0.02
+    max_gripper_step:=0.002
+    mujoco_headless:=false
     joint_state_topic_hardware:=false
     joint_commands_topic:=/joint_commands_topic
@@ -20,5 +26,5 @@
           <param name="mujoco_model">$(find piper_mujoco)/models/piper.xml</param>
           <param name="use_sim_time">true</param>
-          <param name="headless">false</param>
+          <param name="headless">${mujoco_headless}</param>
         </xacro:if>
         <!-- This supports Isaac sim and Hardware -->
@@ -30,5 +36,4 @@
         <xacro:if value="${mock_hardware}">
           <plugin>mock_components/GenericSystem</plugin>
-          <param name="fake_sensor_commands">${fake_sensor_commands}</param>
           <param name="state_following_offset">0.0</param>
         </xacro:if>
@@ -36,10 +41,16 @@
         <xacro:if value="${real_hardware}">
           <plugin>piper_control/PiperHardware</plugin>
+          <param name="can_interface">${can_interface}</param>
+          <param name="calibration_mode">${calibration_mode}</param>
+          <param name="speed_percent">${speed_percent}</param>
+          <param name="feedback_timeout_ms">${feedback_timeout_ms}</param>
+          <param name="max_arm_step">${max_arm_step}</param>
+          <param name="max_gripper_step">${max_gripper_step}</param>
         </xacro:if>
       </hardware>
       <joint name="${prefix}joint1">
         <command_interface name="position">
-          <param name="min">-2.618</param>
-          <param name="max">2.618</param>
+          <param name="min">-2.6179</param>
+          <param name="max">2.6179</param>
         </command_interface>
         <state_interface name="position">
@@ -54,5 +65,5 @@
         <command_interface name="position">
           <param name="min">0.0</param>
-          <param name="max">${pi}</param>
+          <param name="max">3.14</param>
         </command_interface>
         <state_interface name="position">
@@ -79,6 +90,6 @@
       <joint name="${prefix}joint4">
         <command_interface name="position">
-          <param name="min">-1.832</param>
-          <param name="max">1.832</param>
+          <param name="min">-1.745</param>
+          <param name="max">1.745</param>
         </command_interface>
         <state_interface name="position">
@@ -105,6 +116,6 @@
       <joint name="${prefix}joint6">
         <command_interface name="position">
-          <param name="min">-${pi}</param>
-          <param name="max">${pi}</param>
+          <param name="min">-2.09439</param>
+          <param name="max">2.09439</param>
         </command_interface>
         <state_interface name="position">
@@ -118,5 +129,8 @@
       <xacro:if value="${include_gripper}">
         <joint name="${prefix}gripper_joint">
-          <command_interface name="position"/>
+          <command_interface name="position">
+            <param name="min">0.0</param>
+            <param name="max">0.035</param>
+          </command_interface>
           <state_interface name="position">
             <param name="initial_value">0.0</param>

File: src/piper_description/urdf/piper.urdf.xacro (robot description, xacro)
@@ -7,4 +7,11 @@
     <xacro:arg name="mock_hardware" default="false" />
     <xacro:arg name="real_hardware" default="false" />
+    <xacro:arg name="calibration_mode" default="false" />
+    <xacro:arg name="can_interface" default="can0" />
+    <xacro:arg name="speed_percent" default="20" />
+    <xacro:arg name="feedback_timeout_ms" default="250" />
+    <xacro:arg name="max_arm_step" default="0.02" />
+    <xacro:arg name="max_gripper_step" default="0.002" />
+    <xacro:arg name="mujoco_headless" default="false" />
     <!-- Import macros for main hardware components -->
     <xacro:include filename="$(find piper_description)/urdf/piper_macro.xacro" />
@@ -43,4 +50,11 @@
         sim_mujoco="$(arg sim_mujoco)"
         real_hardware="$(arg real_hardware)"
+        calibration_mode="$(arg calibration_mode)"
+        can_interface="$(arg can_interface)"
+        speed_percent="$(arg speed_percent)"
+        feedback_timeout_ms="$(arg feedback_timeout_ms)"
+        max_arm_step="$(arg max_arm_step)"
+        max_gripper_step="$(arg max_gripper_step)"
+        mujoco_headless="$(arg mujoco_headless)"
         initial_positions="${xacro.load_yaml(initial_positions_file)}">
       <origin xyz="0 0 0" rpy="0 0 0" />  <!-- position robot in the world -->

File: src/piper_description/urdf/piper_arm_macro.xacro (robot description, xacro)
@@ -61,5 +61,5 @@
       <child link="${prefix}link_1" />
       <axis xyz="0 0 1" />
-      <limit lower="-2.68" upper="2.68" effort="100" velocity="3.14" />
+      <limit lower="-2.6179" upper="2.6179" effort="100" velocity="0.8" />
     </joint>
     <link name="${prefix}link_2">
@@ -91,5 +91,5 @@
       <child link="${prefix}link_2" />
       <axis xyz="0 0 1" />
-      <limit lower="0" upper="3.4" effort="100" velocity="3.4" />
+      <limit lower="0" upper="3.14" effort="100" velocity="0.8" />
     </joint>
     <link name="${prefix}link_3">
@@ -121,5 +121,5 @@
       <child link="${prefix}link_3" />
       <axis xyz="0 0 1" />
-      <limit lower="-2.697" upper="0" effort="100" velocity="3.14" />
+      <limit lower="-2.697" upper="0" effort="100" velocity="0.8" />
     </joint>
     <link name="${prefix}link_4">
@@ -151,5 +151,5 @@
       <child link="${prefix}link_4" />
       <axis xyz="0 0 1" />
-      <limit lower="-1.85" upper="1.85" effort="100" velocity="3.93" />
+      <limit lower="-1.745" upper="1.745" effort="100" velocity="0.8" />
     </joint>
     <link name="${prefix}link_5">
@@ -181,5 +181,5 @@
       <child link="${prefix}link_5" />
       <axis xyz="0 0 1" />
-      <limit lower="-1.3" upper="1.3" effort="100" velocity="3.93" />
+      <limit lower="-1.22" upper="1.22" effort="100" velocity="0.8" />
     </joint>
     <link name="${prefix}link_6">
@@ -210,5 +210,5 @@
       <child link="${prefix}link_6" />
       <axis xyz="0 0 1" />
-      <limit lower="-${pi}" upper="${pi}" effort="100" velocity="3.93" />
+      <limit lower="-2.09439" upper="2.09439" effort="100" velocity="0.8" />
     </joint>
     <link name="${prefix}tool_0" />

File: src/piper_description/urdf/piper_gripper_macro.xacro (robot description, xacro)
@@ -26,5 +26,5 @@
       <child link="${prefix}left_finger"/>
       <axis xyz="0 0 -1" />
-      <limit lower="0" upper="0.035" effort="20" velocity="0.1" />
+      <limit lower="0" upper="0.035" effort="20" velocity="0.08" />
     </joint>
     <link name="${prefix}left_finger">
@@ -57,5 +57,5 @@
       <child link="${prefix}right_finger"/>
       <axis xyz="0 0 1" />
-      <limit lower="-0.035" upper="0" effort="20" velocity="0.1" />
+      <limit lower="-0.035" upper="0" effort="20" velocity="0.08" />
       <mimic joint="${prefix}gripper_joint" multiplier="-1" offset="0" />
     </joint>

File: src/piper_description/urdf/piper_macro.xacro (robot description, xacro)
@@ -12,4 +12,11 @@
     mock_hardware:=true
     real_hardware:=false
+    calibration_mode:=false
+    can_interface:=can0
+    speed_percent:=20
+    feedback_timeout_ms:=250
+    max_arm_step:=0.02
+    max_gripper_step:=0.002
+    mujoco_headless:=false
     initial_positions:=${dict(joint1=0.0,joint2=0.0,joint3=0.0,joint4=0.0,joint5=0.0,joint6=0.0)}">
     <xacro:include filename="$(find piper_description)/urdf/piper_arm_macro.xacro" />
@@ -36,4 +43,11 @@
       mock_hardware="${mock_hardware}"
       real_hardware="${real_hardware}"
+      calibration_mode="${calibration_mode}"
+      can_interface="${can_interface}"
+      speed_percent="${speed_percent}"
+      feedback_timeout_ms="${feedback_timeout_ms}"
+      max_arm_step="${max_arm_step}"
+      max_gripper_step="${max_gripper_step}"
+      mujoco_headless="${mujoco_headless}"
       sim_mujoco="${sim_mujoco}"
       joint_commands_topic="${joint_commands_topic}"

File: src/piper_moveit_config/config/piper.srdf.xacro (robot description, xacro)
@@ -82,12 +82,5 @@
     <disable_collisions link1="gripper_base_link" link2="right_finger" reason="Adjacent"/>
     <disable_collisions link1="left_finger" link2="right_finger" reason="Default"/>
-    <!-- 禁用 table 与所有其他 link 的碰撞 -->
-    <disable_collisions link1="table" link2="link_2" reason="Never"/>
-    <disable_collisions link1="table" link2="link_3" reason="Never"/>
-    <disable_collisions link1="table" link2="link_4" reason="Never"/>
-    <disable_collisions link1="table" link2="link_5" reason="Never"/>
-    <disable_collisions link1="table" link2="link_6" reason="Never"/>
-    <disable_collisions link1="table" link2="gripper_base_link" reason="Never"/>
-    <disable_collisions link1="table" link2="left_finger" reason="Never"/>
-    <disable_collisions link1="table" link2="right_finger" reason="Never"/>
+    <!-- Only the mounted base/first link may overlap the table model. Distal
+         arm and gripper links deliberately keep table collision checking. -->
 </robot>
